File: Kicad PCB/comp-test/comp-test.kicad_sch (KiCad schematic)
At the start: 26 parts

Commit message: Added Schematic PDF
Parts:
- gave numbers to parts that had none: 26
Other:
- title: (none) -> Component Tester
